Commit message: add sensors

File: my_robot/urdf/my_robot.xacro (robot description, xacro)
@@ -55,3 +55,123 @@
     </visual>
   </link>
+  <link name="left_wheel">
+    <inertial>
+      <mass value="5.0"/>
+      <origin xyz="0.0 0 0" rpy=" 0 1.5707 1.5707"/>
+      <inertia
+          ixx="0.1" ixy="0" ixz="0"
+          iyy="0.1" iyz="0"
+          izz="0.1"
+      />
+    </inertial>
+    <collision name='collision'>
+      <origin xyz="0 0 0" rpy=" 0 1.5707 1.5707"/>
+      <geometry>
+        <cylinder radius="0.1" length = "0.05"/>
+      </geometry>
+    </collision>
+    <visual name='left_wheel_visual'>
+      <origin xyz="0 0 0" rpy=" 0 1.5707 1.5707"/>
+      <geometry>
+        <cylinder radius="0.1" length = "0.05"/>
+      </geometry>
+    </visual>
+  </link>
+  <link name="right_wheel">
+    <inertial>
+      <mass value="5.0"/>
+      <origin xyz="0.0 0 0" rpy=" 0 1.5707 1.5707"/>
+      <inertia
+          ixx="0.1" ixy="0" ixz="0"
+          iyy="0.1" iyz="0"
+          izz="0.1"
+      />
+    </inertial>
+    <collision name='collision'>
+      <origin xyz="0 0 0" rpy=" 0 1.5707 1.5707"/>
+      <geometry>
+        <cylinder radius="0.1" length = "0.05"/>
+      </geometry>
+    </collision>
+    <visual name='left_wheel_visual'>
+      <origin xyz="0 0 0" rpy=" 0 1.5707 1.5707"/>
+      <geometry>
+        <cylinder radius="0.1" length = "0.05"/>
+      </geometry>
+    </visual>
+  </link>
+  <joint type="continuous" name="left_wheel_hinge">
+    <origin xyz="0 0.15 0" rpy="0 0 0"/>
+    <child link="left_wheel"/>
+    <parent link="chassis"/>
+    <axis xyz="0 1 0" rpy="0 0 0"/>
+    <limit effort="10000" velocity="1000"/>
+    <dynamics damping="1.0" friction="1.0"/>
+  </joint>
+  <joint type="continuous" name="right_wheel_hinge">
+    <origin xyz="0 -0.15 0" rpy="0 0 0"/>
+    <child link="right_wheel"/>
+    <parent link="chassis"/>
+    <axis xyz="0 1 0" rpy="0 0 0"/>
+    <limit effort="10000" velocity="1000"/>
+    <dynamics damping="1.0" friction="1.0"/>
+  </joint>
+  <link name="camera">
+    <inertial>
+      <mass value="0.1"/>
+      <origin xyz="0.0 0 0" rpy=" 0 0 0"/>
+      <inertia
+          ixx="1e-6" ixy="0" ixz="0"
+          iyy="1e-6" iyz="0"
+          izz="1e-6"
+      />
+    </inertial>
+    <collision name='collision'>
+      <origin xyz="0.0 0 0" rpy=" 0 0 0"/>
+      <geometry>
+         <box size=".05 .05 .05"/>
+      </geometry>
+    </collision>
+    <visual name='camera_visual'>
+      <origin xyz="0.0 0 0" rpy=" 0 0 0"/>
+      <geometry>
+         <box size=".05 .05 .05"/>
+      </geometry>
+    </visual>
+  </link>
+  <joint type="fixed" name="camera_joint">
+    <origin xyz="0.2 0 0" rpy="0 0 0"/>
+    <child link="camera"/>
+    <parent link="chassis"/>
+    <axis xyz="0 1 0" rpy="0 0 0"/>
+  </joint>
+  <link name="hokuyo">
+    <inertial>
+      <mass value="1e-5"/>
+      <origin xyz="0 0 0" rpy=" 0 0 0"/>
+      <inertia
+          ixx="1e-6" ixy="0" ixz="0"
+          iyy="1e-6" iyz="0"
+          izz="1e-6"
+      />
+    </inertial>
+    <collision name='collision'>
+      <origin xyz="0 0 0" rpy=" 0 0 0"/>
+      <geometry>
+         <box size=".1 .1 .1"/>
+      </geometry>
+    </collision>
+    <visual name='hokuyo_visual'>
+      <origin xyz="0 0 0" rpy=" 0 0 0"/>
+      <geometry>
+         <mesh filename="package://my_robot/meshes/hokuyo.dae"/>
+      </geometry>
+    </visual>
+  </link>
+  <joint type="fixed" name="hokuyo_joint">
+    <origin xyz="0.15 0 0.1" rpy="0 0 0"/>
+    <child link="hokuyo"/>
+    <parent link="chassis"/>
+    <axis xyz="0 1 0" rpy="0 0 0"/>
+  </joint>
 </robot>

Commit message: skid steer wip

File: my_robot/urdf/my_robot.xacro (robot description, xacro)
@@ -2,4 +2,23 @@
 <robot name="my_robot" xmlns:xacro="http://www.ros.org/wiki/xacro">
   <xacro:include filename="$(find my_robot)/urdf/my_robot.gazebo" />
+  <xacro:property name="chassis_width" value="0.35" />
+  <xacro:property name="chassis_length" value="0.45" />
+  <xacro:property name="chassis_height" value="0.1" />
+  <xacro:property name="chassis_mass" value="5" />
+  <xacro:property name="chassis_ixx" value="${chassis_mass/12.0 * (chassis_height*chassis_height + chassis_width*chassis_width)}" />
+  <xacro:property name="chassis_iyy" value="${chassis_mass/12.0 * (chassis_height*chassis_height + chassis_length*chassis_length)}" />
+  <xacro:property name="chassis_izz" value="${chassis_mass/12.0 * (chassis_width*chassis_width + chassis_length*chassis_length)}" />
+  <xacro:property name="wheel_length" value="0.05" />
+  <xacro:property name="wheel_radius" value="0.1" />
+  <xacro:property name="wheel_mass" value="1" />
+  <xacro:property name="wheel_inertia" value="0.1" />
+  <!-- <xacro:property name="wheel_x_offset" value="${base_x_offset + mower_length/2.0}" />
+  <xacro:property name="wheel_y_offset" value="${mower_width/2.0 - wheel_length/2.0}" /> -->
+  <xacro:property name="wheel_kp" value="100.0" />
+  <xacro:property name="wheel_kd" value="1.0" />
+  <xacro:property name="wheel_mu1" value="1000" />
+  <xacro:property name="wheel_mu2" value="1000" />
+  <xacro:property name="wheel_slip1" value="0" />
+  <xacro:property name="wheel_slip2" value="0" />
   <link name="robot_footprint"></link>
   <joint name="robot_footprint_joint" type="fixed">
@@ -11,16 +30,16 @@
     <pose>0 0 0.1 0 0 0</pose>
     <inertial>
-      <mass value="15.0"/>
-      <origin xyz="0.0 0 0" rpy=" 0 0 0"/>
-      <inertia
-          ixx="0.1" ixy="0" ixz="0"
-          iyy="0.1" iyz="0"
-          izz="0.1"
-      />
-    </inertial>
-    <collision name='collision'>
-      <origin xyz="0 0 0" rpy=" 0 0 0"/>
-      <geometry>
-        <box size=".4 .2 .1"/>
+      <mass value="${chassis_mass}"/>
+      <origin xyz="0.0 0 0" rpy=" 0 0 0"/>
+      <inertia
+          ixx="${chassis_ixx}" ixy="0" ixz="0"
+          iyy="${chassis_iyy}" iyz="0"
+          izz="${chassis_izz}"
+      />
+    </inertial>
+    <collision name='collision'>
+      <origin xyz="0 0 0" rpy=" 0 0 0"/>
+      <geometry>
+        <box size="${chassis_length} ${chassis_width} ${chassis_height}"/>
       </geometry>
     </collision>
@@ -28,89 +47,171 @@
       <origin xyz="0 0 0" rpy=" 0 0 0"/>
       <geometry>
-        <box size=".4 .2 .1"/>
-      </geometry>
-    </visual>
-    <collision name='back_caster_collision'>
-      <origin xyz="-0.15 0 -0.05" rpy=" 0 0 0"/>
-      <geometry>
-        <sphere radius="0.0499"/>
-      </geometry>
-    </collision>
-    <visual name='back_caster_visual'>
-      <origin xyz="-0.15 0 -0.05" rpy=" 0 0 0"/>
-      <geometry>
-        <sphere radius="0.05"/>
-      </geometry>
-    </visual>
-    <collision name='front_caster_collision'>
-      <origin xyz="0.15 0 -0.05" rpy=" 0 0 0"/>
-      <geometry>
-        <sphere radius="0.0499"/>
-      </geometry>
-    </collision>
-    <visual name='front_caster_visual'>
-      <origin xyz="0.15 0 -0.05" rpy=" 0 0 0"/>
-      <geometry>
-        <sphere radius="0.05"/>
-      </geometry>
-    </visual>
-  </link>
-  <link name="left_wheel">
-    <inertial>
-      <mass value="5.0"/>
-      <origin xyz="0.0 0 0" rpy=" 0 1.5707 1.5707"/>
-      <inertia
-          ixx="0.1" ixy="0" ixz="0"
-          iyy="0.1" iyz="0"
-          izz="0.1"
-      />
-    </inertial>
-    <collision name='collision'>
-      <origin xyz="0 0 0" rpy=" 0 1.5707 1.5707"/>
-      <geometry>
-        <cylinder radius="0.1" length = "0.05"/>
-      </geometry>
-    </collision>
-    <visual name='left_wheel_visual'>
-      <origin xyz="0 0 0" rpy=" 0 1.5707 1.5707"/>
-      <geometry>
-        <cylinder radius="0.1" length = "0.05"/>
-      </geometry>
-    </visual>
-  </link>
-  <link name="right_wheel">
-    <inertial>
-      <mass value="5.0"/>
-      <origin xyz="0.0 0 0" rpy=" 0 1.5707 1.5707"/>
-      <inertia
-          ixx="0.1" ixy="0" ixz="0"
-          iyy="0.1" iyz="0"
-          izz="0.1"
-      />
-    </inertial>
-    <collision name='collision'>
-      <origin xyz="0 0 0" rpy=" 0 1.5707 1.5707"/>
-      <geometry>
-        <cylinder radius="0.1" length = "0.05"/>
-      </geometry>
-    </collision>
-    <visual name='left_wheel_visual'>
-      <origin xyz="0 0 0" rpy=" 0 1.5707 1.5707"/>
-      <geometry>
-        <cylinder radius="0.1" length = "0.05"/>
-      </geometry>
-    </visual>
-  </link>
-  <joint type="continuous" name="left_wheel_hinge">
-    <origin xyz="0 0.15 0" rpy="0 0 0"/>
-    <child link="left_wheel"/>
-    <parent link="chassis"/>
-    <axis xyz="0 1 0" rpy="0 0 0"/>
-    <limit effort="10000" velocity="1000"/>
-    <dynamics damping="1.0" friction="1.0"/>
-  </joint>
-  <joint type="continuous" name="right_wheel_hinge">
-    <origin xyz="0 -0.15 0" rpy="0 0 0"/>
-    <child link="right_wheel"/>
+        <box size="${chassis_length} ${chassis_width} ${chassis_height}"/>
+      </geometry>
+    </visual>
+  </link>
+  <link name="left_front_wheel">
+    <inertial>
+      <mass value="${wheel_mass}"/>
+      <origin xyz="0.0 0 0" rpy=" 0 1.5707 1.5707"/>
+      <inertia
+          ixx="${wheel_inertia}" ixy="0" ixz="0"
+          iyy="${wheel_inertia}" iyz="0"
+          izz="${wheel_inertia}"
+      />
+    </inertial>
+    <collision name='collision'>
+      <origin xyz="0 0 0" rpy=" 0 1.5707 1.5707"/>
+      <geometry>
+        <cylinder radius="${wheel_radius}" length = "${wheel_length}"/>
+      </geometry>
+      <surface>
+        <friction>
+          <fdir1>1 0 0</fdir1>
+          <kp>${wheel_kp}</kp> <!-- kp and kd for rubber -->
+          <kd>${wheel_kd}</kd>
+          <mu>${wheel_mu1}</mu>
+          <mu2>${wheel_mu2}</mu2>
+          <slip1>${wheel_slip1}</slip1>
+          <slip2>${wheel_slip2}</slip2>
+        </friction>
+      </surface>
+    </collision>
+    <visual name='left_front_wheel_visual'>
+      <origin xyz="0 0 0" rpy=" 0 1.5707 1.5707"/>
+      <geometry>
+        <cylinder radius="${wheel_radius}" length = "${wheel_length}"/>
+      </geometry>
+    </visual>
+  </link>
+  <link name="left_rear_wheel">
+    <inertial>
+      <mass value="${wheel_mass}"/>
+      <origin xyz="0.0 0 0" rpy=" 0 1.5707 1.5707"/>
+      <inertia
+          ixx="${wheel_inertia}" ixy="0" ixz="0"
+          iyy="${wheel_inertia}" iyz="0"
+          izz="${wheel_inertia}"
+      />
+    </inertial>
+    <collision name='collision'>
+      <origin xyz="0 0 0" rpy=" 0 1.5707 1.5707"/>
+      <geometry>
+        <cylinder radius="${wheel_radius}" length = "${wheel_length}"/>
+      </geometry>
+      <surface>
+        <friction>
+          <fdir1>1 0 0</fdir1>
+          <kp>${wheel_kp}</kp> <!-- kp and kd for rubber -->
+          <kd>${wheel_kd}</kd>
+          <mu>${wheel_mu1}</mu>
+          <mu2>${wheel_mu2}</mu2>
+          <slip1>${wheel_slip1}</slip1>
+          <slip2>${wheel_slip2}</slip2>
+        </friction>
+      </surface>
+    </collision>
+    <visual name='left_rear_wheel_visual'>
+      <origin xyz="0 0 0" rpy=" 0 1.5707 1.5707"/>
+      <geometry>
+        <cylinder radius="${wheel_radius}" length = "${wheel_length}"/>
+      </geometry>
+    </visual>
+  </link>
+  <link name="right_front_wheel">
+    <inertial>
+      <mass value="${wheel_mass}"/>
+      <origin xyz="0.0 0 0" rpy=" 0 1.5707 1.5707"/>
+      <inertia
+          ixx="${wheel_inertia}" ixy="0" ixz="0"
+          iyy="${wheel_inertia}" iyz="0"
+          izz="${wheel_inertia}"
+      />
+    </inertial>
+    <collision name='collision'>
+      <origin xyz="0 0 0" rpy=" 0 1.5707 1.5707"/>
+      <geometry>
+        <cylinder radius="${wheel_radius}" length = "${wheel_length}"/>
+      </geometry>
+      <surface>
+        <friction>
+          <fdir1>1 0 0</fdir1>
+          <kp>${wheel_kp}</kp> <!-- kp and kd for rubber -->
+          <kd>${wheel_kd}</kd>
+          <mu>${wheel_mu1}</mu>
+          <mu2>${wheel_mu2}</mu2>
+          <slip1>${wheel_slip1}</slip1>
+          <slip2>${wheel_slip2}</slip2>
+        </friction>
+      </surface>
+    </collision>
+    <visual name='right_front_wheel_visual'>
+      <origin xyz="0 0 0" rpy=" 0 1.5707 1.5707"/>
+      <geometry>
+        <cylinder radius="${wheel_radius}" length = "${wheel_length}"/>
+      </geometry>
+    </visual>
+  </link>
+  <link name="right_rear_wheel">
+    <inertial>
+      <mass value="${wheel_mass}"/>
+      <origin xyz="0.0 0 0" rpy=" 0 1.5707 1.5707"/>
+      <inertia
+          ixx="${wheel_inertia}" ixy="0" ixz="0"
+          iyy="${wheel_inertia}" iyz="0"
+          izz="${wheel_inertia}"
+      />
+    </inertial>
+    <collision name='collision'>
+      <origin xyz="0 0 0" rpy=" 0 1.5707 1.5707"/>
+      <geometry>
+        <cylinder radius="${wheel_radius}" length = "${wheel_length}"/>
+      </geometry>
+      <surface>
+        <friction>
+          <fdir1>1 0 0</fdir1>
+          <kp>${wheel_kp}</kp> <!-- kp and kd for rubber -->
+          <kd>${wheel_kd}</kd>
+          <mu>${wheel_mu1}</mu>
+          <mu2>${wheel_mu2}</mu2>
+          <slip1>${wheel_slip1}</slip1>
+          <slip2>${wheel_slip2}</slip2>
+        </friction>
+      </surface>
+    </collision>
+    <visual name='right_rear_wheel_visual'>
+      <origin xyz="0 0 0" rpy=" 0 1.5707 1.5707"/>
+      <geometry>
+        <cylinder radius="${wheel_radius}" length = "${wheel_length}"/>
+      </geometry>
+    </visual>
+  </link>
+  <joint type="continuous" name="left_front_wheel_hinge">
+    <origin xyz="0.11 ${chassis_width/2+wheel_length/2} 0" rpy="0 0 0"/>
+    <child link="left_front_wheel"/>
+    <parent link="chassis"/>
+    <axis xyz="0 1 0" rpy="0 0 0"/>
+    <limit effort="10000" velocity="1000"/>
+    <dynamics damping="1.0" friction="1.0"/>
+  </joint>
+  <joint type="continuous" name="right_front_wheel_hinge">
+    <origin xyz="0.11 -${chassis_width/2+wheel_length/2} 0" rpy="0 0 0"/>
+    <child link="right_front_wheel"/>
+    <parent link="chassis"/>
+    <axis xyz="0 1 0" rpy="0 0 0"/>
+    <limit effort="10000" velocity="1000"/>
+    <dynamics damping="1.0" friction="1.0"/>
+  </joint>
+  <joint type="continuous" name="left_rear_wheel_hinge">
+    <origin xyz="-0.11 ${chassis_width/2+wheel_length/2} 0" rpy="0 0 0"/>
+    <child link="left_rear_wheel"/>
+    <parent link="chassis"/>
+    <axis xyz="0 1 0" rpy="0 0 0"/>
+    <limit effort="10000" velocity="1000"/>
+    <dynamics damping="1.0" friction="1.0"/>
+  </joint>
+  <joint type="continuous" name="right_rear_wheel_hinge">
+    <origin xyz="-0.11 -${chassis_width/2+wheel_length/2} 0" rpy="0 0 0"/>
+    <child link="right_rear_wheel"/>
     <parent link="chassis"/>
     <axis xyz="0 1 0" rpy="0 0 0"/>
@@ -142,5 +243,5 @@
   </link>
   <joint type="fixed" name="camera_joint">
-    <origin xyz="0.2 0 0" rpy="0 0 0"/>
+    <origin xyz="0.225 0 0" rpy="0 0 0"/>
     <child link="camera"/>
     <parent link="chassis"/>
@@ -171,5 +272,5 @@
   </link>
   <joint type="fixed" name="hokuyo_joint">
-    <origin xyz="0.15 0 0.1" rpy="0 0 0"/>
+    <origin xyz="0.0 0 0.1" rpy="0 0 0"/>
     <child link="hokuyo"/>
     <parent link="chassis"/>

Commit message: update robot

File: my_robot/urdf/my_robot.xacro (robot description, xacro)
@@ -2,8 +2,8 @@
 <robot name="my_robot" xmlns:xacro="http://www.ros.org/wiki/xacro">
   <xacro:include filename="$(find my_robot)/urdf/my_robot.gazebo" />
-  <xacro:property name="chassis_width" value="0.35" />
+  <xacro:property name="chassis_width" value="0.2" />
   <xacro:property name="chassis_length" value="0.45" />
   <xacro:property name="chassis_height" value="0.1" />
-  <xacro:property name="chassis_mass" value="5" />
+  <xacro:property name="chassis_mass" value="15" />
   <xacro:property name="chassis_ixx" value="${chassis_mass/12.0 * (chassis_height*chassis_height + chassis_width*chassis_width)}" />
   <xacro:property name="chassis_iyy" value="${chassis_mass/12.0 * (chassis_height*chassis_height + chassis_length*chassis_length)}" />
@@ -11,14 +11,7 @@
   <xacro:property name="wheel_length" value="0.05" />
   <xacro:property name="wheel_radius" value="0.1" />
-  <xacro:property name="wheel_mass" value="1" />
+  <xacro:property name="wheel_mass" value="5" />
   <xacro:property name="wheel_inertia" value="0.1" />
-  <!-- <xacro:property name="wheel_x_offset" value="${base_x_offset + mower_length/2.0}" />
-  <xacro:property name="wheel_y_offset" value="${mower_width/2.0 - wheel_length/2.0}" /> -->
-  <xacro:property name="wheel_kp" value="100.0" />
-  <xacro:property name="wheel_kd" value="1.0" />
-  <xacro:property name="wheel_mu1" value="1000" />
-  <xacro:property name="wheel_mu2" value="1000" />
-  <xacro:property name="wheel_slip1" value="0" />
-  <xacro:property name="wheel_slip2" value="0" />
+  <xacro:property name="wheel_offset" value="0.15" />
   <link name="robot_footprint"></link>
   <joint name="robot_footprint_joint" type="fixed">
@@ -66,15 +59,4 @@
         <cylinder radius="${wheel_radius}" length = "${wheel_length}"/>
       </geometry>
-      <surface>
-        <friction>
-          <fdir1>1 0 0</fdir1>
-          <kp>${wheel_kp}</kp> <!-- kp and kd for rubber -->
-          <kd>${wheel_kd}</kd>
-          <mu>${wheel_mu1}</mu>
-          <mu2>${wheel_mu2}</mu2>
-          <slip1>${wheel_slip1}</slip1>
-          <slip2>${wheel_slip2}</slip2>
-        </friction>
-      </surface>
     </collision>
     <visual name='left_front_wheel_visual'>
@@ -100,15 +82,4 @@
         <cylinder radius="${wheel_radius}" length = "${wheel_length}"/>
       </geometry>
-      <surface>
-        <friction>
-          <fdir1>1 0 0</fdir1>
-          <kp>${wheel_kp}</kp> <!-- kp and kd for rubber -->
-          <kd>${wheel_kd}</kd>
-          <mu>${wheel_mu1}</mu>
-          <mu2>${wheel_mu2}</mu2>
-          <slip1>${wheel_slip1}</slip1>
-          <slip2>${wheel_slip2}</slip2>
-        </friction>
-      </surface>
     </collision>
     <visual name='left_rear_wheel_visual'>
@@ -134,15 +105,4 @@
         <cylinder radius="${wheel_radius}" length = "${wheel_length}"/>
       </geometry>
-      <surface>
-        <friction>
-          <fdir1>1 0 0</fdir1>
-          <kp>${wheel_kp}</kp> <!-- kp and kd for rubber -->
-          <kd>${wheel_kd}</kd>
-          <mu>${wheel_mu1}</mu>
-          <mu2>${wheel_mu2}</mu2>
-          <slip1>${wheel_slip1}</slip1>
-          <slip2>${wheel_slip2}</slip2>
-        </friction>
-      </surface>
     </collision>
     <visual name='right_front_wheel_visual'>
@@ -168,15 +128,4 @@
         <cylinder radius="${wheel_radius}" length = "${wheel_length}"/>
       </geometry>
-      <surface>
-        <friction>
-          <fdir1>1 0 0</fdir1>
-          <kp>${wheel_kp}</kp> <!-- kp and kd for rubber -->
-          <kd>${wheel_kd}</kd>
-          <mu>${wheel_mu1}</mu>
-          <mu2>${wheel_mu2}</mu2>
-          <slip1>${wheel_slip1}</slip1>
-          <slip2>${wheel_slip2}</slip2>
-        </friction>
-      </surface>
     </collision>
     <visual name='right_rear_wheel_visual'>
@@ -188,5 +137,5 @@
   </link>
   <joint type="continuous" name="left_front_wheel_hinge">
-    <origin xyz="0.11 ${chassis_width/2+wheel_length/2} 0" rpy="0 0 0"/>
+    <origin xyz="0.11 ${wheel_offset} 0" rpy="0 0 0"/>
     <child link="left_front_wheel"/>
     <parent link="chassis"/>
@@ -196,5 +145,5 @@
   </joint>
   <joint type="continuous" name="right_front_wheel_hinge">
-    <origin xyz="0.11 -${chassis_width/2+wheel_length/2} 0" rpy="0 0 0"/>
+    <origin xyz="0.11 -${wheel_offset} 0" rpy="0 0 0"/>
     <child link="right_front_wheel"/>
     <parent link="chassis"/>
@@ -204,5 +153,5 @@
   </joint>
   <joint type="continuous" name="left_rear_wheel_hinge">
-    <origin xyz="-0.11 ${chassis_width/2+wheel_length/2} 0" rpy="0 0 0"/>
+    <origin xyz="-0.11 ${wheel_offset} 0" rpy="0 0 0"/>
     <child link="left_rear_wheel"/>
     <parent link="chassis"/>
@@ -212,5 +161,5 @@
   </joint>
   <joint type="continuous" name="right_rear_wheel_hinge">
-    <origin xyz="-0.11 -${chassis_width/2+wheel_length/2} 0" rpy="0 0 0"/>
+    <origin xyz="-0.11 -${wheel_offset} 0" rpy="0 0 0"/>
     <child link="right_rear_wheel"/>
     <parent link="chassis"/>
@@ -221,5 +170,5 @@
   <link name="camera">
     <inertial>
-      <mass value="0.1"/>
+      <mass value="1e-5"/>
       <origin xyz="0.0 0 0" rpy=" 0 0 0"/>
       <inertia
